Commit message: add pydrake for learning

File: drake_controller/spot.urdf (robot description, URDF)
Before this commit: robot spot, 13 links, 12 joints
Links:
- link base: geometry collision mesh filename=link_models/base.obj; visual mesh filename=link_models/base.obj
- link fl.lleg: geometry collision mesh filename=link_models/fl.lleg.obj; visual mesh filename=link_models/fl.lleg.obj
- link fr.lleg: geometry collision mesh filename=link_models/fr.lleg.obj; visual mesh filename=link_models/fr.lleg.obj
- link hl.lleg: geometry collision mesh filename=link_models/hl.lleg.obj; visual mesh filename=link_models/hl.lleg.obj
- link hr.lleg: geometry collision mesh filename=link_models/hr.lleg.obj; visual mesh filename=link_models/hr.lleg.obj

Commit message: add doc

File: drake_controller/spot.urdf (robot description, URDF)
Before this commit: robot spot, 13 links, 12 joints
Links:
- link fl.hip: mass 2 -> None
- link fl.uleg: mass 1 -> None
- link fr.hip: mass 2 -> None
- link fr.uleg: mass 1 -> None
- link hl.hip: mass 2 -> None
- link hl.uleg: mass 1 -> None
- link hr.hip: mass 2 -> None
- link hr.uleg: mass 1 -> None
